File: hardware/KiCad Main Board/Power.kicad_sch (KiCad schematic)
At the start: 51 parts, among them J9 Batt_Conn, Q2 AO3401A, Q3 AO3400A, Q4 AO3400A, Q5 AO3400A, Q6 AO3400A, U10 LM5157RTER, U2 S-8252ACP-M6T1U, U4 AP63203WU, U9 MCP73844-820I/MS

Commit message: changed some footprints and minor routing changes
Parts:
- L3: footprint Inductor_SMD:L_APV_APH0650 -> Inductor_SMD_Wurth:L_Wurth_WE-LQSH-4020
Changed lines of the file:
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@@
 			)
 		)
-		(property "Footprint" "Inductor_SMD:L_APV_APH0650"
+		(property "Footprint" "Inductor_SMD_Wurth:L_Wurth_WE-LQSH-4020"
 			(at 113.03 21.59 0)
 			(effects

Commit message: changing charging circuitry because the current regulater is linear
Parts:
- added C101, C73, C75: 4.7u, Capacitor_SMD:C_0603_1608Metric_Pad1.08x0.95mm_HandSolder, symbol Device:C_Small
- added D60: B340, Diode_SMD:D_SMA, symbol Diode:B340
- added J10: Batt_Conn, TestPoint:TestPoint_2Pads_Pitch2.54mm_Drill0.8mm, symbol Connector:Conn_01x02_Pin
- added R53: 27k, Resistor_SMD:R_0603_1608Metric_Pad0.98x0.95mm_HandSolder, symbol Device:R_Small
- added R55, R57, R58, R59: 5k1, Resistor_SMD:R_0603_1608Metric_Pad0.98x0.95mm_HandSolder, symbol Device:R_Small
- added R56: 0, Resistor_SMD:R_0603_1608Metric_Pad0.98x0.95mm_HandSolder, symbol Device:R_Small
- added R60: 10k, Resistor_SMD:R_0603_1608Metric_Pad0.98x0.95mm_HandSolder, symbol Device:R_Small
- added U3: MP2672GD-0000-Z, QFN-18_2MMx3MM_MP2672_MNP_MPS, symbol MP2672GD:MP2672GD-0000-Z
Connections:
- net 5V_USB: now also D60.2 (A)
- net GND: now also C101.2, C73.2, C75.2, J10.1 (Pin_1), R55.1, R58.2, R59.1, U3.13 (PGND), U3.6 (AGND); no longer J9.1 (Pin_1)
- net V_BAT_RAW: now also C101.1, C75.1, U3.11 (SYS); no longer J9.2 (Pin_2), TP30.1
- net V_CHG: no longer TP5.1
- new net: R53.1, R55.2
- new net: C73.1, D60.1 (K), R60.2, TP5.1, U3.1 (IN)
- new net: J10.2 (Pin_2), TP30.1, U3.10 (BATT)
- new net: R53.2, R56.1, U3.17 (CV)
- new net: R56.2, U3.4 (VCC)
- new net: R57.1, U3.5 (ISET)
- new net: R59.2, R60.1, U3.7 (VLIM)
- new net: R57.2, R58.1
- new net CHGR_I2C_SCL: U3.14 (SCL)
- new net CHGR_I2C_SDA: U3.15 (SDA)
- no-connect marks 0 -> 1
Other:
- moved on the sheet: J9, TP30, TP5

Commit message: fixed connector in mainboard schematic that I moved accidentally
Connections:
- net GND: now also J9.1 (Pin_1)
- net V_BAT_RAW: now also J9.2 (Pin_2)
Other:
- moved on the sheet: J9
Changed lines of the file:
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@@
 	(symbol
 		(lib_id "Connector:Conn_01x02_Pin")
-		(at 45.497 129.9651 90)
+		(at 179.07 99.06 180)
 		(unit 1)
 		(exclude_from_sim no)
@@
 		(fields_autoplaced yes)
 		(property "Reference" "J9"
-			(at 50.577 128.06 90)
+			(at 180.34 96.5199 0)
 			(effects
 				(font
@@
 		)
 		(property "Value" "Batt_Conn"
-			(at 50.577 130.6 90)
+			(at 180.34 99.0599 0)
 			(effects
 				(font
@@
 		)
 		(property "Footprint" "TestPoint:TestPoint_2Pads_Pitch2.54mm_Drill0.8mm"
-			(at 45.497 129.9651 0)
+			(at 179.07 99.06 0)
 			(effects
 				(font
@@
 		)
 		(property "Datasheet" "~"
-			(at 45.497 129.9651 0)
+			(at 179.07 99.06 0)
 			(effects
 				(font
@@
 		)
 		(property "Description" "Generic connector, single row, 01x02, script generated"
-			(at 45.497 129.9651 0)
+			(at 179.07 99.06 0)
 			(effects
 				(font
